File: PCB/opendtu.sch (EAGLE design)
At the start: 11 parts, among them M1 DISPLAY-OLED-128X64-I2CNH, M3 NRF24L01-PA-EXT, X1 MCV1,5/2G

Commit message: Schematic
Schaltplan änderungen
Other:
- note added: "Florian Schoop"
Changed lines of the file:
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@@
 IO22 SCL
 IO21 SDA</text>
+<text x="226.06" y="7.62" size="2.54" layer="91" ratio="15">Florian Schoop</text>
 </plain>
 <instances>

Commit message: Gerber V1.1
V1.1 vom Gerber
Other:
- note added: "5V Eingang mini combicon"
- note added: "Display Versorungsspannung J1 1-2 1+ J2 2-3 1- J2 1-2 2- J2 2-3 2+ Achtung verpolungs gefahr !"
- note removed: "Display Versorungsspannung J1 1-2 1+ J2 2-3 1- J2 1-2 2- J2 2-3 2+ Achtung Kurzschluss gefahr !"
Changed lines of the file:
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@@
 J1  1-2  1+       J2 2-3  1-
 J2  1-2  2-        J2 2-3  2+
-Achtung Kurzschluss gefahr !</text>
+Achtung verpolungs gefahr !</text>
 <text x="170.18" y="167.64" size="2.54" layer="91" ratio="15">Display 90°</text>
 <text x="10.16" y="7.62" size="2.54" layer="91" ratio="15">OpenDTU
@@
 IO21 SDA</text>
 <text x="226.06" y="7.62" size="2.54" layer="91" ratio="15">Florian Schoop</text>
+<text x="58.42" y="99.06" size="2.54" layer="91" ratio="15">5V Eingang
+mini combicon</text>
 </plain>
 <instances>
