File: PCB/opendtu V2.brd (EAGLE design)
At the start: 104.1 x 54 mm, 12 parts, among them M1 DISPLAY-OLED-128X64-I2CNH, M3 NRF24L01-PA-EXT, X1 MCV1,5/2G

Commit message: plus war im weg
plus war im weg
Parts:
- moved C1 0.63 mm to (71.8, 8.89)
Routing:
- net +3.3V: track 158.7 -> 159.3 mm
Changed lines of the file:
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@@
 <element name="J1" library="jumper_fs" package="SJ_2" value="" x="50.165" y="46.99" rot="MR0"/>
 <element name="J2" library="jumper_fs" package="SJ_2" value="" x="67.31" y="46.99" rot="MR0"/>
-<element name="C1" library="5elko" package="EB10D" value="470uF" x="71.12" y="8.89" rot="R270"/>
+<element name="C1" library="5elko" package="EB10D" value="470uF" x="71.755" y="8.89" rot="R270"/>
 <element name="X1" library="STECKER" package="MCV1,5/2" value="MCV1,5/2G" x="35.56" y="8.255" rot="R270"/>
 <element name="ESP32" library="wemos d1" package="WEMOS-ESP32" value="WEMOS-ESP32" x="10.795" y="14.605"/>
@@
 <contactref element="ESP32" pad="3V3"/>
 <contactref element="U$11" pad="3.3V"/>
-<wire x1="62.865" y1="46.99" x2="51.689" y2="46.99" width="0.8128" layer="16"/>
+<wire x1="64.135" y1="46.99" x2="51.689" y2="46.99" width="0.8128" layer="16"/>
 <wire x1="66.04" y1="46.99" x2="65.786" y2="46.99" width="0.4064" layer="16"/>
 <wire x1="13.335" y1="26.035" x2="15.24" y2="26.035" width="0.8128" layer="16"/>
@@
 <wire x1="17.145" y1="24.13" x2="17.145" y2="17.78" width="0.8128" layer="16"/>
 <wire x1="17.145" y1="17.78" x2="17.78" y2="17.145" width="0.8128" layer="16"/>
-<wire x1="45.72" y1="13.335" x2="48.26" y2="13.335" width="0.8128" layer="16"/>
-<wire x1="69.215" y1="13.335" x2="71.12" y2="11.43" width="0.8128" layer="16"/>
+<wire x1="44.45" y1="13.335" x2="48.26" y2="13.335" width="0.8128" layer="16"/>
 <wire x1="91.44" y1="24.765" x2="90.17" y2="23.495" width="0.8128" layer="16"/>
 <wire x1="90.17" y1="23.495" x2="69.85" y2="23.495" width="0.8128" layer="16"/>
@@
 <wire x1="69.85" y1="23.495" x2="69.215" y2="24.13" width="0.8128" layer="1"/>
 <wire x1="69.215" y1="24.13" x2="69.215" y2="38.1" width="0.8128" layer="1"/>
-<wire x1="69.215" y1="38.1" x2="62.865" y2="44.45" width="0.8128" layer="1"/>
-<wire x1="62.865" y1="44.45" x2="62.865" y2="46.99" width="0.8128" layer="1"/>
-<via x="62.865" y="46.99" extent="1-16" drill="0.6"/>
-<wire x1="62.865" y1="46.99" x2="65.786" y2="46.99" width="0.8128" layer="16"/>
+<wire x1="64.135" y1="44.45" x2="64.135" y2="46.99" width="0.8128" layer="1"/>
+<via x="64.135" y="46.99" extent="1-16" drill="0.6"/>
+<wire x1="64.135" y1="46.99" x2="65.786" y2="46.99" width="0.8128" layer="16"/>
 <wire x1="48.26" y1="17.01" x2="48.26" y2="18.415" width="0.4064" layer="1"/>
 <via x="48.26" y="18.415" extent="1-16" drill="0.6"/>
@@
 <wire x1="17.78" y1="17.145" x2="40.64" y2="17.145" width="0.8128" layer="16"/>
 <wire x1="40.64" y1="17.145" x2="44.45" y2="13.335" width="0.8128" layer="16"/>
-<wire x1="44.45" y1="13.335" x2="45.72" y2="13.335" width="0.8128" layer="16"/>
+<wire x1="69.215" y1="38.1" x2="64.135" y2="44.45" width="0.8128" layer="1"/>
+<wire x1="69.215" y1="13.335" x2="71.12" y2="13.335" width="0.8128" layer="16"/>
+<wire x1="71.12" y1="13.335" x2="71.755" y2="12.7" width="0.8128" layer="16"/>
+<wire x1="71.755" y1="12.7" x2="71.755" y2="11.43" width="0.8128" layer="16"/>
 </signal>
 <signal name="CE">
