File: PCB/opendtu V2.sch (EAGLE design)
At the start: 12 parts, among them M1 DISPLAY-OLED-128X64-I2CNH, M3 NRF24L01-PA-EXT, X1 MCV1,5/2G

Commit message: Schaltplan PDF
Other:
- note added: "OpenDTU Wemos D1 ESP GPIO Belegung NRF: IO17 IRQ IO16 CE IO5 CS IO23 MOSI IO19 MISO IO18 SCK Display: IO22 SCL IO21 SDA CMT2300a: IO14 SDIO IO12 SCLK IO27 CSN IO26 FCSB IO04 GPIO2 IO13 GPIO3 LED: IO32 LED0 IO33 LED1"
- note removed: "OpenDTU Wemos D1 ESP GPIO Belegung IO17 IRQ IO16 CE IO5 CS IO23 MOSI IO19 MISO IO18 SCK IO22 SCL IO21 SDA"
Changed lines of the file:
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@@
 J2  1-2  2-        J2 2-3  2+
 Achtung verpolungs gefahr !</text>
-<text x="10.16" y="7.62" size="2.54" layer="91" ratio="15">OpenDTU
+<text x="238.76" y="50.8" size="2.54" layer="91" ratio="15">OpenDTU
 Wemos D1 ESP
 GPIO Belegung
+NRF:
 IO17 IRQ
 IO16 CE
@@
 IO19 MISO
 IO18 SCK
+Display:
 IO22 SCL
-IO21 SDA</text>
+IO21 SDA
+CMT2300a:
+IO14 SDIO
+IO12 SCLK
+IO27 CSN
+IO26 FCSB
+IO04 GPIO2
+IO13 GPIO3
+LED:
+IO32 LED0
+IO33 LED1</text>
 <text x="226.06" y="7.62" size="2.54" layer="91" ratio="15">Florian Schoop</text>
 <text x="170.18" y="34.29" size="2.54" layer="91" ratio="15">5V Eingang

Commit message: Bezeichnung korrigiert
Beschreibung J1 und J2 im Schaltplan war falsch.
Other:
- note added: "Display Versorungsspannung J1 1-2 1+ J1 2-3 1- J2 1-2 2- J2 2-3 2+ Achtung verpolungs Gefahr !"
- note removed: "Display Versorungsspannung J1 1-2 1+ J2 2-3 1- J2 1-2 2- J2 2-3 2+ Achtung verpolungs gefahr !"
Changed lines of the file:
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@@
 <plain>
 <text x="97.79" y="167.64" size="2.54" layer="91" ratio="15">Display Versorungsspannung
-J1  1-2  1+       J2 2-3  1-
+J1  1-2  1+       J1 2-3  1-
 J2  1-2  2-        J2 2-3  2+
-Achtung verpolungs gefahr !</text>
+Achtung verpolungs Gefahr !</text>
 <text x="238.76" y="50.8" size="2.54" layer="91" ratio="15">OpenDTU
 Wemos D1 ESP
